File: 2024/KiCad Projects/AQ-SAO/AQ-SAO.kicad_pcb (KiCad board)
At the start: 2 copper layers, 50.8 x 25.4 mm, 13 parts, among them J1 SAO (on back), U1 74HC00, U2 74HC00

Commit message: Updating KiCad PCB files and README
Parts:
- removed GND: GND, TestPoint:TestPoint_THTPad_1.0x1.0mm_Drill0.5mm
- removed SCL: SCL, TestPoint:TestPoint_THTPad_1.0x1.0mm_Drill0.5mm
- removed SDA: SDA, TestPoint:TestPoint_THTPad_1.0x1.0mm_Drill0.5mm
- removed VCC: VCC, TestPoint:TestPoint_THTPad_1.0x1.0mm_Drill0.5mm
- added H1: MountingHole, MountingHole:MountingHole_2.2mm_M2, F.Cu at (57.1, 53.3)
- added H2: MountingHole, MountingHole:MountingHole_2.2mm_M2, F.Cu at (74.9, 53.3)
- added H3: MountingHole, MountingHole:MountingHole_2.2mm_M2, F.Cu at (57.1, 73.7)
- added H4: MountingHole, MountingHole:MountingHole_2.2mm_M2, F.Cu at (74.9, 73.7)
- added J2: SDA-SCL, Connector_PinHeader_2.54mm:PinHeader_1x02_P2.54mm_Vertical, F.Cu at (60.0, 66.8)
- added J3: VCC-GND, Connector_PinHeader_2.54mm:PinHeader_1x02_P2.54mm_Vertical, F.Cu at (60.0, 60.3)
- moved J1 1.27 mm to (56.0, 61.0)
Routing:
- net Net-(J1-Pin_3): track 11.2 -> 5.35 mm
- net Net-(J1-Pin_6): track 39.8 -> 44.4 mm
- net Net-(J1-Pin_5): track 39.2 -> 43.5 mm
- net Net-(J1-Pin_4): track 8.15 -> 9.46 mm
Other:
- outline, holes or cut-outs redrawn
- board text added: "GND"
- board text added: "SCL"
- board text added: "SDA"
- board text added: "VCC"
